File: gpio.sch (KiCad schematic (older format))
At the start: 13 parts, among them J20 Rain, J21 GPIO, J22 Wind, U4 PCA9536D

Commit message: Added images Added information to schematic Added information to layout
Parts:
- renumbered C27 to C23, C28 to C24, C29 to C25, J20 to J16, J21 to J17, J22 to J18
Changed lines of the file:
@@
 encoding utf-8
 Sheet 9 11
-Title ""
-Date ""
-Rev ""
-Comp ""
-Comment1 ""
+Title "AirMon"
+Date "2020-01-13"
+Rev "0.1"
+Comp "Jörg Bayer"
+Comment1 "CC BY 4.0"
 Comment2 ""
 Comment3 ""
@@
 AR Path="/5E1991ED/5E1CF5AA" Ref="#PWR?"  Part="1"
 AR Path="/5E1C55BA/5E1CF5AA" Ref="#PWR?"  Part="1"
-AR Path="/5E1CBADF/5E1CF5AA" Ref="#PWR039"  Part="1"
-F 0 "#PWR039" H 4900 2850 50  0001 C CNN
+AR Path="/5E1CBADF/5E1CF5AA" Ref="#PWR034"  Part="1"
+F 0 "#PWR034" H 4900 2850 50  0001 C CNN
 F 1 "VSS" H 4800 3100 50  0000 C CNN
 F 2 "" H 4900 3000 50  0001 C CNN
@@
 AR Path="/5E151517/5E298533" Ref="C?"  Part="1"
 AR Path="/5E1991ED/5E298533" Ref="C?"  Part="1"
-AR Path="/5E1CBADF/5E298533" Ref="C27"  Part="1"
-F 0 "C27" H 5615 1496 50  0000 L CNN
+AR Path="/5E1CBADF/5E298533" Ref="C23"  Part="1"
+F 0 "C23" H 5615 1496 50  0000 L CNN
 F 1 "1u" H 5615 1405 50  0000 L CNN
 F 2 "Capacitor_SMD:C_0805_2012Metric" H 5538 1300 50  0001 C CNN
@@
 AR Path="/5E151517/5E29895C" Ref="C?"  Part="1"
 AR Path="/5E1991ED/5E29895C" Ref="C?"  Part="1"
-AR Path="/5E1CBADF/5E29895C" Ref="C28"  Part="1"
-F 0 "C28" H 5915 1896 50  0000 L CNN
+AR Path="/5E1CBADF/5E29895C" Ref="C24"  Part="1"
+F 0 "C24" H 5915 1896 50  0000 L CNN
 F 1 "1u" H 5915 1805 50  0000 L CNN
 F 2 "Capacitor_SMD:C_0805_2012Metric" H 5838 1700 50  0001 C CNN
@@
 AR Path="/5E151517/5E1E9685" Ref="C?"  Part="1"
 AR Path="/5E1EC3C1/5E1E9685" Ref="C?"  Part="1"
-AR Path="/5E1CBADF/5E1E9685" Ref="C29"  Part="1"
-F 0 "C29" H 7015 1896 50  0000 L CNN
+AR Path="/5E1CBADF/5E1E9685" Ref="C25"  Part="1"
+F 0 "C25" H 7015 1896 50  0000 L CNN
 F 1 "100n" H 7015 1805 50  0000 L CNN
 F 2 "Capacitor_SMD:C_0603_1608Metric" H 6938 1700 50  0001 C CNN
@@
 AR Path="/5E1991ED/5E1EA209" Ref="#PWR?"  Part="1"
 AR Path="/5E1C55BA/5E1EA209" Ref="#PWR?"  Part="1"
-AR Path="/5E1CBADF/5E1EA209" Ref="#PWR044"  Part="1"
-F 0 "#PWR044" H 7300 2950 50  0001 C CNN
+AR Path="/5E1CBADF/5E1EA209" Ref="#PWR039"  Part="1"
+F 0 "#PWR039" H 7300 2950 50  0001 C CNN
 F 1 "VSS" H 7200 3200 50  0000 C CNN
 F 2 "" H 7300 3100 50  0001 C CNN
@@
 AR Path="/5E1991ED/5E1EB394" Ref="#PWR?"  Part="1"
 AR Path="/5E1C55BA/5E1EB394" Ref="#PWR?"  Part="1"
-AR Path="/5E1CBADF/5E1EB394" Ref="#PWR042"  Part="1"
-F 0 "#PWR042" H 6900 1950 50  0001 C CNN
+AR Path="/5E1CBADF/5E1EB394" Ref="#PWR037"  Part="1"
+F 0 "#PWR037" H 6900 1950 50  0001 C CNN
 F 1 "VSS" H 6800 2200 50  0000 C CNN
 F 2 "" H 6900 2100 50  0001 C CNN
@@
 AR Path="/5E198729/5E1F09A8" Ref="#PWR?"  Part="1"
 AR Path="/5E1C55BA/5E1F09A8" Ref="#PWR?"  Part="1"
-AR Path="/5E1CBADF/5E1F09A8" Ref="#PWR043"  Part="1"
-F 0 "#PWR043" H 7300 1350 50  0001 C CNN
+AR Path="/5E1CBADF/5E1F09A8" Ref="#PWR038"  Part="1"
+F 0 "#PWR038" H 7300 1350 50  0001 C CNN
 F 1 "VCC" H 7317 1673 50  0000 C CNN
 F 2 "" H 7300 1500 50  0001 C CNN
@@
 GPIO_6
 $Comp
-L Connector:RJ12 J20
+L Connector:RJ12 J16
 U 1 1 5E205904
 P 3900 3700
-F 0 "J20" V 3909 4130 50  0000 L CNN
+F 0 "J16" V 3909 4130 50  0000 L CNN
 F 1 "Rain" V 4000 4130 50  0000 L CNN
 F 2 "global:DS1133-S60" V 3900 3725 50  0001 C CNN
@@
 AR Path="/5E1991ED/5E20AC6D" Ref="#PWR?"  Part="1"
 AR Path="/5E1C55BA/5E20AC6D" Ref="#PWR?"  Part="1"
-AR Path="/5E1CBADF/5E20AC6D" Ref="#PWR038"  Part="1"
-F 0 "#PWR038" H 3900 4150 50  0001 C CNN
+AR Path="/5E1CBADF/5E20AC6D" Ref="#PWR033"  Part="1"
+F 0 "#PWR033" H 3900 4150 50  0001 C CNN
 F 1 "VSS" H 3800 4400 50  0000 C CNN
 F 2 "" H 3900 4300 50  0001 C CNN
@@
 AR Path="/5E198729/5E212762" Ref="#PWR?"  Part="1"
 AR Path="/5E1C55BA/5E212762" Ref="#PWR?"  Part="1"
-AR Path="/5E1CBADF/5E212762" Ref="#PWR040"  Part="1"
-F 0 "#PWR040" H 4900 3250 50  0001 C CNN
+AR Path="/5E1CBADF/5E212762" Ref="#PWR035"  Part="1"
+F 0 "#PWR035" H 4900 3250 50  0001 C CNN
 F 1 "VCC" H 4917 3573 50  0000 C CNN
 F 2 "" H 4900 3400 50  0001 C CNN
@@
 A1
 $Comp
-L Connector:RJ12 J22
+L Connector:RJ12 J18
 U 1 1 5E2192FF
 P 5900 3700
-F 0 "J22" V 5909 4130 50  0000 L CNN
+F 0 "J18" V 5909 4130 50  0000 L CNN
 F 1 "Wind" V 6000 4130 50  0000 L CNN
 F 2 "global:DS1133-S60" V 5900 3725 50  0001 C CNN
@@
 AR Path="/5E1991ED/5E21C2C5" Ref="#PWR?"  Part="1"
 AR Path="/5E1C55BA/5E21C2C5" Ref="#PWR?"  Part="1"
-AR Path="/5E1CBADF/5E21C2C5" Ref="#PWR041"  Part="1"
-F 0 "#PWR041" H 6100 4150 50  0001 C CNN
+AR Path="/5E1CBADF/5E21C2C5" Ref="#PWR036"  Part="1"
+F 0 "#PWR036" H 6100 4150 50  0001 C CNN
 F 1 "VSS" H 6000 4400 50  0000 C CNN
 F 2 "" H 6100 4300 50  0001 C CNN
@@
 GPIO_2
 $Comp
-L Connector_Generic:Conn_02x06_Odd_Even J21
+L Connector_Generic:Conn_02x06_Odd_Even J17
 U 1 1 5E259AAF
 P 4800 2300
-F 0 "J21" H 4850 2817 50  0000 C CNN
+F 0 "J17" H 4850 2817 50  0000 C CNN
 F 1 "GPIO" H 4850 2726 50  0000 C CNN
 F 2 "Connector_PinHeader_2.54mm:PinHeader_2x06_P2.54mm_Vertical" H 4800 2300 50  0001 C CNN

Commit message: Added fuse for USB Added buttons for boot and reset Added version number to PCB Changed several component values for improved manufacturing Added BOM Added component position file
Parts:
- C23, C24: lcsc# (none) -> C28323; manf# CL21B105KBFNNNG -> CL21B105KBFNNNE
- C25: lcsc# (none) -> C14663; manf# CL10B104KB8NNNL -> CC0603KRX7R9BB104
- J16, J18: lcsc# (none) -> C77856
- R20, R22: lcsc# (none) -> C23162; manf# (none) -> 0603WAF4701T5E
- R21: lcsc# (none) -> C25804; manf# (none) -> 0603WAF1002T5E
- U4: lcsc# (none) -> C129522; manf# (none) -> PCA9536D
Changed lines of the file:
@@
 F 2 "Capacitor_SMD:C_0805_2012Metric" H 5538 1300 50  0001 C CNN
 F 3 "~" H 5500 1450 50  0001 C CNN
-F 4 "CL21B105KBFNNNG" H 5500 1450 50  0001 C CNN "manf#"
+F 4 "CL21B105KBFNNNE" H 5500 1450 50  0001 C CNN "manf#"
+F 5 "C28323" H 0   0   50  0001 C CNN "lcsc#"
 	1    5500 1450
 	1    0    0    -1
@@
 F 2 "Capacitor_SMD:C_0805_2012Metric" H 5838 1700 50  0001 C CNN
 F 3 "~" H 5800 1850 50  0001 C CNN
-F 4 "CL21B105KBFNNNG" H 5800 1850 50  0001 C CNN "manf#"
+F 4 "CL21B105KBFNNNE" H 5800 1850 50  0001 C CNN "manf#"
+F 5 "C28323" H 0   0   50  0001 C CNN "lcsc#"
 	1    5800 1850
 	1    0    0    -1
@@
 F 2 "Package_SO:SOIC-8_3.9x4.9mm_P1.27mm" H 8300 2150 50  0001 C CNN
 F 3 "http://www.nxp.com/documents/data_sheet/PCA9536.pdf" H 7100 800 50  0001 C CNN
+F 4 "C129522" H 0   0   50  0001 C CNN "lcsc#"
+F 5 "PCA9536D" H 0   0   50  0001 C CNN "manf#"
 	1    7300 2500
 	1    0    0    -1
@@
 F 2 "Capacitor_SMD:C_0603_1608Metric" H 6938 1700 50  0001 C CNN
 F 3 "~" H 6900 1850 50  0001 C CNN
-F 4 "CL10B104KB8NNNL" H 6900 1850 50  0001 C CNN "manf#"
+F 4 "CC0603KRX7R9BB104" H 6900 1850 50  0001 C CNN "manf#"
+F 5 "C14663" H 0   0   50  0001 C CNN "lcsc#"
 	1    6900 1850
 	1    0    0    -1
@@
 F 3 "~" V 3900 3725 50  0001 C CNN
 F 4 "DS1133-S40BPX" V 3900 3700 50  0001 C CNN "manf#"
+F 5 "C77856" H 0   0   50  0001 C CNN "lcsc#"
 	1    3900 3700
 	0    1    1    0
@@
 F 2 "Resistor_SMD:R_0603_1608Metric" V 4530 3750 50  0001 C CNN
 F 3 "~" H 4600 3750 50  0001 C CNN
+F 4 "C23162" H 0   0   50  0001 C CNN "lcsc#"
+F 5 "0603WAF4701T5E" H 0   0   50  0001 C CNN "manf#"
 	1    4600 3750
 	-1   0    0    -1
@@
 F 3 "~" V 5900 3725 50  0001 C CNN
 F 4 "DS1133-S40BPX" V 5900 3700 50  0001 C CNN "manf#"
+F 5 "C77856" H 0   0   50  0001 C CNN "lcsc#"
 	1    5900 3700
 	0    1    1    0
@@
 F 2 "Resistor_SMD:R_0603_1608Metric" V 4830 3750 50  0001 C CNN
 F 3 "~" H 4900 3750 50  0001 C CNN
+F 4 "C25804" H 0   0   50  0001 C CNN "lcsc#"
+F 5 "0603WAF1002T5E" H 0   0   50  0001 C CNN "manf#"
 	1    4900 3750
 	-1   0    0    -1
@@
 F 2 "Resistor_SMD:R_0603_1608Metric" V 5130 3750 50  0001 C CNN
 F 3 "~" H 5200 3750 50  0001 C CNN
+F 4 "C23162" H 0   0   50  0001 C CNN "lcsc#"
+F 5 "0603WAF4701T5E" H 0   0   50  0001 C CNN "manf#"
 	1    5200 3750
 	-1   0    0    -1

Commit message: Moved to KiCad 5.1.5_3
Parts:
- U4: symbol Interface_Expansion:PCA9536D -> airMon-rescue:PCA9536D-Interface_Expansion
Changed lines of the file:
@@
 EESchema Schematic File Version 4
-LIBS:airMon-cache
-EELAYER 26 0
+EELAYER 30 0
 EELAYER END
 $Descr A4 11693 8268
@@
 Connection ~ 4500 1300
 $Comp
-L Interface_Expansion:PCA9536D U4
+L airMon-rescue:PCA9536D-Interface_Expansion U4
 U 1 1 5E1E8043
 P 7300 2500

Commit message: Added RFM95 Module for Lora Added Changelog Changed input voltage monitoring from A2(IO35) to A3(IO36) Removed A3 12V compatibility Rearranged IOs to fit new components
Connections:
- net LORA_RST: now reaches U4.5 (IO3)
- no-connect marks 7 -> 6
Changed lines of the file:
@@
 $Descr A4 11693 8268
 encoding utf-8
-Sheet 9 11
+Sheet 9 12
 Title "AirMon"
 Date "2020-01-17"
@@
 Wire Wire Line
 	4400 1700 5200 1700
-NoConn ~ 7800 2700
+Wire Wire Line
+	7800 2700 8000 2700
+Text HLabel 8000 2700 2    50   Output ~ 0
+LORA_RST
 $EndSCHEMATC
