File: i2c_1.sch (KiCad schematic (older format))
At the start: 6 parts, among them J6 I2C_1_1, J8 I2C_1_2

Commit message: Added images Added information to schematic Added information to layout
Parts:
- renumbered C11 to C10, J6 to J7
Changed lines of the file:
@@
 encoding utf-8
 Sheet 5 11
-Title ""
-Date ""
-Rev ""
-Comp ""
-Comment1 ""
+Title "AirMon"
+Date "2020-01-13"
+Rev "0.1"
+Comp "Jörg Bayer"
+Comment1 "CC BY 4.0"
 Comment2 ""
 Comment3 ""
@@
 $EndDescr
 $Comp
-L Connector_Generic:Conn_01x04 J6
+L Connector_Generic:Conn_01x04 J7
 U 1 1 5E1988DE
 P 4600 2300
-F 0 "J6" H 4680 2292 50  0000 L CNN
+F 0 "J7" H 4680 2292 50  0000 L CNN
 F 1 "I2C_1_1" H 4680 2201 50  0000 L CNN
 F 2 "Connector_PinSocket_2.54mm:PinSocket_1x04_P2.54mm_Vertical" H 4600 2300 50  0001 C CNN
@@
 AR Path="/5E151517/5E1989A5" Ref="#PWR?"  Part="1"
 AR Path="/5E1961BA/5E1989A5" Ref="#PWR?"  Part="1"
-AR Path="/5E198729/5E1989A5" Ref="#PWR012"  Part="1"
-F 0 "#PWR012" H 4300 1850 50  0001 C CNN
+AR Path="/5E198729/5E1989A5" Ref="#PWR014"  Part="1"
+F 0 "#PWR014" H 4300 1850 50  0001 C CNN
 F 1 "VCC" H 4317 2173 50  0000 C CNN
 F 2 "" H 4300 2000 50  0001 C CNN
@@
 AR Path="/5E151517/5E1989AB" Ref="#PWR?"  Part="1"
 AR Path="/5E1961BA/5E1989AB" Ref="#PWR?"  Part="1"
-AR Path="/5E198729/5E1989AB" Ref="#PWR013"  Part="1"
-F 0 "#PWR013" H 4300 2550 50  0001 C CNN
+AR Path="/5E198729/5E1989AB" Ref="#PWR015"  Part="1"
+F 0 "#PWR015" H 4300 2550 50  0001 C CNN
 F 1 "VSS" H 4200 2800 50  0000 C CNN
 F 2 "" H 4300 2700 50  0001 C CNN
@@
 AR Path="/5E15DEC3/5E1AC56F" Ref="C?"  Part="1"
 AR Path="/5E151517/5E1AC56F" Ref="C?"  Part="1"
-AR Path="/5E198729/5E1AC56F" Ref="C11"  Part="1"
-F 0 "C11" H 6815 2396 50  0000 L CNN
+AR Path="/5E198729/5E1AC56F" Ref="C10"  Part="1"
+F 0 "C10" H 6815 2396 50  0000 L CNN
 F 1 "1u" H 6815 2305 50  0000 L CNN
 F 2 "Capacitor_SMD:C_0805_2012Metric" H 6738 2200 50  0001 C CNN

Commit message: Added fuse for USB Added buttons for boot and reset Added version number to PCB Changed several component values for improved manufacturing Added BOM Added component position file
Parts:
- C10, C9: lcsc# (none) -> C28323; manf# CL21B105KBFNNNG -> CL21B105KBFNNNE
- R5, R6: lcsc# (none) -> C23162; manf# (none) -> 0603WAF4701T5E
Changed lines of the file:
@@
 F 2 "Capacitor_SMD:C_0805_2012Metric" H 3338 2200 50  0001 C CNN
 F 3 "~" H 3300 2350 50  0001 C CNN
-F 4 "CL21B105KBFNNNG" H 3300 2350 50  0001 C CNN "manf#"
+F 4 "CL21B105KBFNNNE" H 3300 2350 50  0001 C CNN "manf#"
+F 5 "C28323" H 0   0   50  0001 C CNN "lcsc#"
 	1    3300 2350
 	1    0    0    -1
@@
 F 2 "Capacitor_SMD:C_0805_2012Metric" H 6738 2200 50  0001 C CNN
 F 3 "~" H 6700 2350 50  0001 C CNN
-F 4 "CL21B105KBFNNNG" H 6700 2350 50  0001 C CNN "manf#"
+F 4 "CL21B105KBFNNNE" H 6700 2350 50  0001 C CNN "manf#"
+F 5 "C28323" H 0   0   50  0001 C CNN "lcsc#"
 	1    6700 2350
 	1    0    0    -1
@@
 F 2 "Resistor_SMD:R_0603_1608Metric" V 2830 2450 50  0001 C CNN
 F 3 "~" H 2900 2450 50  0001 C CNN
+F 4 "C23162" H 0   0   50  0001 C CNN "lcsc#"
+F 5 "0603WAF4701T5E" H 0   0   50  0001 C CNN "manf#"
 	1    2900 2450
 	-1   0    0    -1
@@
 F 2 "Resistor_SMD:R_0603_1608Metric" V 2430 2450 50  0001 C CNN
 F 3 "~" H 2500 2450 50  0001 C CNN
+F 4 "C23162" H 0   0   50  0001 C CNN "lcsc#"
+F 5 "0603WAF4701T5E" H 0   0   50  0001 C CNN "manf#"
 	1    2500 2450
 	-1   0    0    -1
