File: i2c_2.sch (KiCad schematic (older format))
At the start: 15 parts, among them J10 I2C_2_1, J11 I2C_2_2, J12 I2C_2_3_Buffer, J13 I2C_2_4_Buffer, U2 P82B715

Commit message: Added images Added information to schematic Added information to layout
Parts:
- renumbered C13 to C11, C14 to C12, C15 to C13, C16 to C14, C17 to C15, C18 to C16, J11 to J10, J12 to J11, J13 to J12, J10 to J9
Changed lines of the file:
@@
 encoding utf-8
 Sheet 6 11
-Title ""
-Date ""
-Rev ""
-Comp ""
-Comment1 ""
+Title "AirMon"
+Date "2020-01-13"
+Rev "0.1"
+Comp "Jörg Bayer"
+Comment1 "CC BY 4.0"
 Comment2 ""
 Comment3 ""
@@
 P 5500 2500
 AR Path="/5E198729/5E199423" Ref="J?"  Part="1"
-AR Path="/5E1991ED/5E199423" Ref="J11"  Part="1"
-F 0 "J11" H 5580 2492 50  0000 L CNN
+AR Path="/5E1991ED/5E199423" Ref="J10"  Part="1"
+F 0 "J10" H 5580 2492 50  0000 L CNN
 F 1 "I2C_2_2" H 5580 2401 50  0000 L CNN
 F 2 "Connector_PinSocket_2.54mm:PinSocket_1x04_P2.54mm_Vertical" H 5500 2500 50  0001 C CNN
@@
 AR Path="/5E1961BA/5E199436" Ref="#PWR?"  Part="1"
 AR Path="/5E198729/5E199436" Ref="#PWR?"  Part="1"
-AR Path="/5E1991ED/5E199436" Ref="#PWR020"  Part="1"
-F 0 "#PWR020" H 5200 2750 50  0001 C CNN
+AR Path="/5E1991ED/5E199436" Ref="#PWR019"  Part="1"
+F 0 "#PWR019" H 5200 2750 50  0001 C CNN
 F 1 "VSS" H 5100 3000 50  0000 C CNN
 F 2 "" H 5200 2900 50  0001 C CNN
@@
 AR Path="/5E1961BA/5E19944D" Ref="#PWR?"  Part="1"
 AR Path="/5E198729/5E19944D" Ref="#PWR?"  Part="1"
-AR Path="/5E1991ED/5E19944D" Ref="#PWR021"  Part="1"
-F 0 "#PWR021" H 8000 1950 50  0001 C CNN
+AR Path="/5E1991ED/5E19944D" Ref="#PWR020"  Part="1"
+F 0 "#PWR020" H 8000 1950 50  0001 C CNN
 F 1 "VCC" H 8017 2273 50  0000 C CNN
 F 2 "" H 8000 2100 50  0001 C CNN
@@
 AR Path="/5E1961BA/5E199453" Ref="#PWR?"  Part="1"
 AR Path="/5E198729/5E199453" Ref="#PWR?"  Part="1"
-AR Path="/5E1991ED/5E199453" Ref="#PWR022"  Part="1"
-F 0 "#PWR022" H 8000 3150 50  0001 C CNN
+AR Path="/5E1991ED/5E199453" Ref="#PWR021"  Part="1"
+F 0 "#PWR021" H 8000 3150 50  0001 C CNN
 F 1 "VSS" H 7900 3400 50  0000 C CNN
 F 2 "" H 8000 3300 50  0001 C CNN
@@
 AR Path="/5E15DEC3/5E19A6BC" Ref="C?"  Part="1"
 AR Path="/5E151517/5E19A6BC" Ref="C?"  Part="1"
-AR Path="/5E1991ED/5E19A6BC" Ref="C14"  Part="1"
-F 0 "C14" H 4415 2596 50  0000 L CNN
+AR Path="/5E1991ED/5E19A6BC" Ref="C12"  Part="1"
+F 0 "C12" H 4415 2596 50  0000 L CNN
 F 1 "1u" H 4415 2505 50  0000 L CNN
 F 2 "Capacitor_SMD:C_0805_2012Metric" H 4338 2400 50  0001 C CNN
@@
 P 10300 2500
 AR Path="/5E198729/5E19E04D" Ref="J?"  Part="1"
-AR Path="/5E1991ED/5E19E04D" Ref="J12"  Part="1"
-F 0 "J12" H 10380 2492 50  0000 L CNN
+AR Path="/5E1991ED/5E19E04D" Ref="J11"  Part="1"
+F 0 "J11" H 10380 2492 50  0000 L CNN
 F 1 "I2C_2_3_Buffer" H 10380 2401 50  0000 L CNN
 F 2 "Connector_PinSocket_2.54mm:PinSocket_1x04_P2.54mm_Vertical" H 10300 2500 50  0001 C CNN
@@
 AR Path="/5E1961BA/5E19E05F" Ref="#PWR?"  Part="1"
 AR Path="/5E198729/5E19E05F" Ref="#PWR?"  Part="1"
-AR Path="/5E1991ED/5E19E05F" Ref="#PWR024"  Part="1"
-F 0 "#PWR024" H 10000 2750 50  0001 C CNN
+AR Path="/5E1991ED/5E19E05F" Ref="#PWR023"  Part="1"
+F 0 "#PWR023" H 10000 2750 50  0001 C CNN
 F 1 "VSS" H 9900 3000 50  0000 C CNN
 F 2 "" H 10000 2900 50  0001 C CNN
@@
 P 10000 2200
 AR Path="/5E18E639/5E1A15D1" Ref="#PWR?"  Part="1"
-AR Path="/5E1991ED/5E1A15D1" Ref="#PWR023"  Part="1"
-F 0 "#PWR023" H 10000 2050 50  0001 C CNN
+AR Path="/5E1991ED/5E1A15D1" Ref="#PWR022"  Part="1"
+F 0 "#PWR022" H 10000 2050 50  0001 C CNN
 F 1 "+5V" H 10015 2373 50  0000 C CNN
 F 2 "" H 10000 2200 50  0001 C CNN
@@
 AR Path="/5E15DEC3/5E1A1CF6" Ref="C?"  Part="1"
 AR Path="/5E151517/5E1A1CF6" Ref="C?"  Part="1"
-AR Path="/5E1991ED/5E1A1CF6" Ref="C17"  Part="1"
-F 0 "C17" H 9715 2396 50  0000 L CNN
+AR Path="/5E1991ED/5E1A1CF6" Ref="C15"  Part="1"
+F 0 "C15" H 9715 2396 50  0000 L CNN
 F 1 "1u" H 9715 2305 50  0000 L CNN
 F 2 "Capacitor_SMD:C_0805_2012Metric" H 9638 2200 50  0001 C CNN
@@
 P 3700 2500
 AR Path="/5E198729/5E1A4C6E" Ref="J?"  Part="1"
-AR Path="/5E1991ED/5E1A4C6E" Ref="J10"  Part="1"
-F 0 "J10" H 3780 2492 50  0000 L CNN
+AR Path="/5E1991ED/5E1A4C6E" Ref="J9"  Part="1"
+F 0 "J9" H 3780 2492 50  0000 L CNN
 F 1 "I2C_2_1" H 3780 2401 50  0000 L CNN
 F 2 "Connector_PinSocket_2.54mm:PinSocket_1x04_P2.54mm_Vertical" H 3700 2500 50  0001 C CNN
@@
 AR Path="/5E1961BA/5E1A4C7A" Ref="#PWR?"  Part="1"
 AR Path="/5E198729/5E1A4C7A" Ref="#PWR?"  Part="1"
-AR Path="/5E1991ED/5E1A4C7A" Ref="#PWR019"  Part="1"
-F 0 "#PWR019" H 3400 2750 50  0001 C CNN
+AR Path="/5E1991ED/5E1A4C7A" Ref="#PWR018"  Part="1"
+F 0 "#PWR018" H 3400 2750 50  0001 C CNN
 F 1 "VSS" H 3300 3000 50  0000 C CNN
 F 2 "" H 3400 2900 50  0001 C CNN
@@
 AR Path="/5E15DEC3/5E1A4C85" Ref="C?"  Part="1"
 AR Path="/5E151517/5E1A4C85" Ref="C?"  Part="1"
-AR Path="/5E1991ED/5E1A4C85" Ref="C13"  Part="1"
-F 0 "C13" H 2615 2596 50  0000 L CNN
+AR Path="/5E1991ED/5E1A4C85" Ref="C11"  Part="1"
+F 0 "C11" H 2615 2596 50  0000 L CNN
 F 1 "1u" H 2615 2505 50  0000 L CNN
 F 2 "Capacitor_SMD:C_0805_2012Metric" H 2538 2400 50  0001 C CNN
@@
 P 3400 2200
 AR Path="/5E18E639/5E1A4C91" Ref="#PWR?"  Part="1"
-AR Path="/5E1991ED/5E1A4C91" Ref="#PWR018"  Part="1"
-F 0 "#PWR018" H 3400 2050 50  0001 C CNN
+AR Path="/5E1991ED/5E1A4C91" Ref="#PWR017"  Part="1"
+F 0 "#PWR017" H 3400 2050 50  0001 C CNN
 F 1 "+5V" H 3415 2373 50  0000 C CNN
 F 2 "" H 3400 2200 50  0001 C CNN
@@
 P 10300 4300
 AR Path="/5E198729/5E1A9AB3" Ref="J?"  Part="1"
-AR Path="/5E1991ED/5E1A9AB3" Ref="J13"  Part="1"
-F 0 "J13" H 10380 4292 50  0000 L CNN
+AR Path="/5E1991ED/5E1A9AB3" Ref="J12"  Part="1"
+F 0 "J12" H 10380 4292 50  0000 L CNN
 F 1 "I2C_2_4_Buffer" H 10380 4201 50  0000 L CNN
 F 2 "Connector_PinSocket_2.54mm:PinSocket_1x04_P2.54mm_Vertical" H 10300 4300 50  0001 C CNN
@@
 AR Path="/5E1961BA/5E1A9ABC" Ref="#PWR?"  Part="1"
 AR Path="/5E198729/5E1A9ABC" Ref="#PWR?"  Part="1"
-AR Path="/5E1991ED/5E1A9ABC" Ref="#PWR025"  Part="1"
-F 0 "#PWR025" H 10000 4550 50  0001 C CNN
+AR Path="/5E1991ED/5E1A9ABC" Ref="#PWR024"  Part="1"
+F 0 "#PWR024" H 10000 4550 50  0001 C CNN
 F 1 "VSS" H 9900 4800 50  0000 C CNN
 F 2 "" H 10000 4700 50  0001 C CNN
@@
 AR Path="/5E15DEC3/5E1A9ACC" Ref="C?"  Part="1"
 AR Path="/5E151517/5E1A9ACC" Ref="C?"  Part="1"
-AR Path="/5E1991ED/5E1A9ACC" Ref="C18"  Part="1"
-F 0 "C18" H 9715 4196 50  0000 L CNN
+AR Path="/5E1991ED/5E1A9ACC" Ref="C16"  Part="1"
+F 0 "C16" H 9715 4196 50  0000 L CNN
 F 1 "1u" H 9715 4105 50  0000 L CNN
 F 2 "Capacitor_SMD:C_0805_2012Metric" H 9638 4000 50  0001 C CNN
@@
 AR Path="/5E15DEC3/5E1ADB5C" Ref="C?"  Part="1"
 AR Path="/5E151517/5E1ADB5C" Ref="C?"  Part="1"
-AR Path="/5E1991ED/5E1ADB5C" Ref="C16"  Part="1"
-F 0 "C16" H 7515 2396 50  0000 L CNN
+AR Path="/5E1991ED/5E1ADB5C" Ref="C14"  Part="1"
+F 0 "C14" H 7515 2396 50  0000 L CNN
 F 1 "100n" H 7515 2305 50  0000 L CNN
 F 2 "Capacitor_SMD:C_0603_1608Metric" H 7438 2200 50  0001 C CNN
@@
 AR Path="/5E15DEC3/5E1B8370" Ref="C?"  Part="1"
 AR Path="/5E151517/5E1B8370" Ref="C?"  Part="1"
-AR Path="/5E1991ED/5E1B8370" Ref="C15"  Part="1"
-F 0 "C15" H 7115 2396 50  0000 L CNN
+AR Path="/5E1991ED/5E1B8370" Ref="C13"  Part="1"
+F 0 "C13" H 7115 2396 50  0000 L CNN
 F 1 "1u" H 7115 2305 50  0000 L CNN
 F 2 "Capacitor_SMD:C_0805_2012Metric" H 7038 2200 50  0001 C CNN

Commit message: Added fuse for USB Added buttons for boot and reset Added version number to PCB Changed several component values for improved manufacturing Added BOM Added component position file
Parts:
- C11, C12, C13, C15, C16: lcsc# (none) -> C28323; manf# CL21B105KBFNNNG -> CL21B105KBFNNNE
- C14: lcsc# (none) -> C14663; manf# CL10B104KB8NNNL -> CC0603KRX7R9BB104
- R10, R9: lcsc# (none) -> C23138; manf# (none) -> 0603WAF3300T5E
- R7, R8: lcsc# (none) -> C23162; manf# (none) -> 0603WAF4701T5E
- U2: digikey# (none) -> 296-24729-1-ND; manf# (none) -> P82B715
Changed lines of the file:
@@
 F 2 "Capacitor_SMD:C_0805_2012Metric" H 4338 2400 50  0001 C CNN
 F 3 "~" H 4300 2550 50  0001 C CNN
-F 4 "CL21B105KBFNNNG" H 4300 2550 50  0001 C CNN "manf#"
+F 4 "CL21B105KBFNNNE" H 4300 2550 50  0001 C CNN "manf#"
+F 5 "C28323" H 0   0   50  0001 C CNN "lcsc#"
 	1    4300 2550
 	1    0    0    -1
@@
 F 2 "Package_SO:SOIC-8_3.9x4.9mm_P1.27mm" H 8000 2700 50  0001 C CNN
 F 3 "http://www.ti.com/lit/ds/symlink/p82b715.pdf" H 8000 2700 50  0001 C CNN
+F 4 "P82B715" H 0   0   50  0001 C CNN "manf#"
+F 5 "	296-24729-1-ND	" H 0   0   50  0001 C CNN "digikey#"
 	1    8000 2700
 	1    0    0    -1
@@
 F 2 "Resistor_SMD:R_0603_1608Metric" V 6530 2350 50  0001 C CNN
 F 3 "~" H 6600 2350 50  0001 C CNN
+F 4 "C23162" H 0   0   50  0001 C CNN "lcsc#"
+F 5 "0603WAF4701T5E" H 0   0   50  0001 C CNN "manf#"
 	1    6600 2350
 	-1   0    0    -1
@@
 F 2 "Resistor_SMD:R_0603_1608Metric" V 6130 2350 50  0001 C CNN
 F 3 "~" H 6200 2350 50  0001 C CNN
+F 4 "C23162" H 0   0   50  0001 C CNN "lcsc#"
+F 5 "0603WAF4701T5E" H 0   0   50  0001 C CNN "manf#"
 	1    6200 2350
 	-1   0    0    -1
@@
 F 2 "Resistor_SMD:R_0603_1608Metric" V 8930 2350 50  0001 C CNN
 F 3 "~" H 9000 2350 50  0001 C CNN
+F 4 "C23138" H 0   0   50  0001 C CNN "lcsc#"
+F 5 "0603WAF3300T5E" H 0   0   50  0001 C CNN "manf#"
 	1    9000 2350
 	-1   0    0    -1
@@
 F 2 "Resistor_SMD:R_0603_1608Metric" V 8530 2350 50  0001 C CNN
 F 3 "~" H 8600 2350 50  0001 C CNN
+F 4 "C23138" H 0   0   50  0001 C CNN "lcsc#"
+F 5 "0603WAF3300T5E" H 0   0   50  0001 C CNN "manf#"
 	1    8600 2350
 	-1   0    0    -1
@@
 F 2 "Capacitor_SMD:C_0805_2012Metric" H 9638 2200 50  0001 C CNN
 F 3 "~" H 9600 2350 50  0001 C CNN
-F 4 "CL21B105KBFNNNG" H 9600 2350 50  0001 C CNN "manf#"
+F 4 "CL21B105KBFNNNE" H 9600 2350 50  0001 C CNN "manf#"
+F 5 "C28323" H 0   0   50  0001 C CNN "lcsc#"
 	1    9600 2350
 	1    0    0    -1
@@
 F 2 "Capacitor_SMD:C_0805_2012Metric" H 2538 2400 50  0001 C CNN
 F 3 "~" H 2500 2550 50  0001 C CNN
-F 4 "CL21B105KBFNNNG" H 2500 2550 50  0001 C CNN "manf#"
+F 4 "CL21B105KBFNNNE" H 2500 2550 50  0001 C CNN "manf#"
+F 5 "C28323" H 0   0   50  0001 C CNN "lcsc#"
 	1    2500 2550
 	1    0    0    -1
@@
 F 2 "Capacitor_SMD:C_0805_2012Metric" H 9638 4000 50  0001 C CNN
 F 3 "~" H 9600 4150 50  0001 C CNN
-F 4 "CL21B105KBFNNNG" H 9600 4150 50  0001 C CNN "manf#"
+F 4 "CL21B105KBFNNNE" H 9600 4150 50  0001 C CNN "manf#"
+F 5 "C28323" H 0   0   50  0001 C CNN "lcsc#"
 	1    9600 4150
 	1    0    0    -1
@@
 F 2 "Capacitor_SMD:C_0603_1608Metric" H 7438 2200 50  0001 C CNN
 F 3 "~" H 7400 2350 50  0001 C CNN
-F 4 "CL10B104KB8NNNL" H 7400 2350 50  0001 C CNN "manf#"
+F 4 "CC0603KRX7R9BB104" H 7400 2350 50  0001 C CNN "manf#"
+F 5 "C14663" H 0   0   50  0001 C CNN "lcsc#"
 	1    7400 2350
 	1    0    0    -1
@@
 F 2 "Capacitor_SMD:C_0805_2012Metric" H 7038 2200 50  0001 C CNN
 F 3 "~" H 7000 2350 50  0001 C CNN
-F 4 "CL21B105KBFNNNG" H 7000 2350 50  0001 C CNN "manf#"
+F 4 "CL21B105KBFNNNE" H 7000 2350 50  0001 C CNN "manf#"
+F 5 "C28323" H 0   0   50  0001 C CNN "lcsc#"
 	1    7000 2350
 	1    0    0    -1
