File: particle.sch (KiCad schematic (older format))
At the start: 6 parts, among them J2 PMS7003, J3 PMSx003, J4 SDS011, J7 Conn_01x05

Commit message: Added images Added information to schematic Added information to layout
Parts:
- renumbered C7 to C6, C4 to C7, J7 to J5
Changed lines of the file:
@@
 encoding utf-8
 Sheet 3 11
-Title ""
-Date ""
-Rev ""
-Comp ""
-Comment1 ""
+Title "AirMon"
+Date "2020-01-13"
+Rev "0.1"
+Comp "Jörg Bayer"
+Comment1 "CC BY 4.0"
 Comment2 ""
 Comment3 ""
@@
 	6700 2200 6700 1600
 $Comp
-L Device:C C7
+L Device:C C6
 U 1 1 5E194A64
 P 4800 1950
-F 0 "C7" H 4915 1996 50  0000 L CNN
+F 0 "C6" H 4915 1996 50  0000 L CNN
 F 1 "10u" H 4915 1905 50  0000 L CNN
 F 2 "Capacitor_SMD:C_1206_3216Metric" H 4838 1800 50  0001 C CNN
@@
 5V_Switched
 $Comp
-L Device:C C4
+L Device:C C7
 U 1 1 5E2321DC
 P 6200 2150
-F 0 "C4" H 6315 2196 50  0000 L CNN
+F 0 "C7" H 6315 2196 50  0000 L CNN
 F 1 "10u" H 6315 2105 50  0000 L CNN
 F 2 "Capacitor_SMD:C_1206_3216Metric" H 6238 2000 50  0001 C CNN
@@
 	5400 2800 5400 2900
 $Comp
-L Connector_Generic:Conn_01x05 J7
+L Connector_Generic:Conn_01x05 J5
 U 1 1 5E1CDC10
 P 8200 2300
-F 0 "J7" H 8280 2342 50  0000 L CNN
+F 0 "J5" H 8280 2342 50  0000 L CNN
 F 1 "Conn_01x05" H 8280 2251 50  0000 L CNN
 F 2 "Connector_JST:JST_XH_B05B-XH-A_1x05_P2.50mm_Vertical" H 8200 2300 50  0001 C CNN
@@
 AR Path="/5E1961BA/5E1CF0A7" Ref="#PWR?"  Part="1"
 AR Path="/5E198729/5E1CF0A7" Ref="#PWR?"  Part="1"
-AR Path="/5E18E639/5E1CF0A7" Ref="#PWR031"  Part="1"
-F 0 "#PWR031" H 8000 1750 50  0001 C CNN
+AR Path="/5E18E639/5E1CF0A7" Ref="#PWR012"  Part="1"
+F 0 "#PWR012" H 8000 1750 50  0001 C CNN
 F 1 "VCC" H 8017 2073 50  0000 C CNN
 F 2 "" H 8000 1900 50  0001 C CNN
@@
 AR Path="/5E15DEC3/5E1CF62F" Ref="#PWR?"  Part="1"
 AR Path="/5E151517/5E1CF62F" Ref="#PWR?"  Part="1"
-AR Path="/5E18E639/5E1CF62F" Ref="#PWR030"  Part="1"
-F 0 "#PWR030" H 7900 2750 50  0001 C CNN
+AR Path="/5E18E639/5E1CF62F" Ref="#PWR011"  Part="1"
+F 0 "#PWR011" H 7900 2750 50  0001 C CNN
 F 1 "VSS" H 7800 3000 50  0000 C CNN
 F 2 "" H 7900 2900 50  0001 C CNN

Commit message: Added fuse for USB Added buttons for boot and reset Added version number to PCB Changed several component values for improved manufacturing Added BOM Added component position file
Parts:
- C6, C7: lcsc# (none) -> C13585; manf# CL31B106KBHNNNE -> CL31A106KBHNNNE
- J3: lcsc# (none) -> C240845; manf# (none) -> 53047-0810
- J4: lcsc# (none) -> C144398; manf# (none) -> B7B-XH-A(LF)(SN)
- J5: lcsc# (none) -> C157991; manf# (none) -> B5B-XH-A(LF)(SN)
Changed lines of the file:
@@
 F 2 "Connector_Molex:Molex_PicoBlade_53047-0810_1x08_P1.25mm_Vertical" H 5700 2300 50  0001 C CNN
 F 3 "~" H 5700 2300 50  0001 C CNN
+F 4 "C240845" H 0   0   50  0001 C CNN "lcsc#"
+F 5 "53047-0810" H 0   0   50  0001 C CNN "manf#"
 	1    5700 2300
 	1    0    0    -1
@@
 F 2 "Connector_JST:JST_XH_B07B-XH-A_1x07_P2.50mm_Vertical" H 7000 2300 50  0001 C CNN
 F 3 "~" H 7000 2300 50  0001 C CNN
+F 4 "C144398" H 0   0   50  0001 C CNN "lcsc#"
+F 5 "B7B-XH-A(LF)(SN)" H 0   0   50  0001 C CNN "manf#"
 	1    7000 2300
 	1    0    0    -1
@@
 F 2 "Capacitor_SMD:C_1206_3216Metric" H 4838 1800 50  0001 C CNN
 F 3 "~" H 4800 1950 50  0001 C CNN
-F 4 "CL31B106KBHNNNE" H 4800 1950 50  0001 C CNN "manf#"
+F 4 "CL31A106KBHNNNE" H 4800 1950 50  0001 C CNN "manf#"
+F 5 "C13585" H 0   0   50  0001 C CNN "lcsc#"
 	1    4800 1950
 	1    0    0    -1
@@
 F 2 "Capacitor_SMD:C_1206_3216Metric" H 6238 2000 50  0001 C CNN
 F 3 "~" H 6200 2150 50  0001 C CNN
-F 4 "CL31B106KBHNNNE" H 6200 2150 50  0001 C CNN "manf#"
+F 4 "CL31A106KBHNNNE" H 6200 2150 50  0001 C CNN "manf#"
+F 5 "C13585" H 0   0   50  0001 C CNN "lcsc#"
 	1    6200 2150
 	1    0    0    -1
@@
 F 2 "Connector_JST:JST_XH_B05B-XH-A_1x05_P2.50mm_Vertical" H 8200 2300 50  0001 C CNN
 F 3 "~" H 8200 2300 50  0001 C CNN
+F 4 "C157991" H 0   0   50  0001 C CNN "lcsc#"
+F 5 "B5B-XH-A(LF)(SN)" H 0   0   50  0001 C CNN "manf#"
 	1    8200 2300
 	1    0    0    1
