File: singleWire.sch (KiCad schematic (older format))
At the start: 3 parts, among them J5 SW

Commit message: Added images Added information to schematic Added information to layout
Parts:
- renumbered J5 to J6
Changed lines of the file:
@@
 encoding utf-8
 Sheet 4 11
-Title ""
-Date ""
-Rev ""
-Comp ""
-Comment1 ""
+Title "AirMon"
+Date "2020-01-13"
+Rev "0.1"
+Comp "Jörg Bayer"
+Comment1 "CC BY 4.0"
 Comment2 ""
 Comment3 ""
@@
 $EndDescr
 $Comp
-L Connector_Generic:Conn_01x04 J5
+L Connector_Generic:Conn_01x04 J6
 U 1 1 5E196217
 P 5400 2700
-F 0 "J5" H 5480 2692 50  0000 L CNN
+F 0 "J6" H 5480 2692 50  0000 L CNN
 F 1 "SW" H 5480 2601 50  0000 L CNN
 F 2 "Connector_PinSocket_2.54mm:PinSocket_1x04_P2.54mm_Vertical" H 5400 2700 50  0001 C CNN
@@
 AR Path="/5E15DEC3/5E198235" Ref="#PWR?"  Part="1"
 AR Path="/5E151517/5E198235" Ref="#PWR?"  Part="1"
-AR Path="/5E1961BA/5E198235" Ref="#PWR011"  Part="1"
-F 0 "#PWR011" H 5100 3050 50  0001 C CNN
+AR Path="/5E1961BA/5E198235" Ref="#PWR013"  Part="1"
+F 0 "#PWR013" H 5100 3050 50  0001 C CNN
 F 1 "VSS" H 5000 3300 50  0000 C CNN
 F 2 "" H 5100 3200 50  0001 C CNN

Commit message: Added fuse for USB Added buttons for boot and reset Added version number to PCB Changed several component values for improved manufacturing Added BOM Added component position file
Parts:
- C8: lcsc# (none) -> C28323; manf# CL21B105KBFNNNG -> CL21B105KBFNNNE
- R4: lcsc# (none) -> C25804; manf# (none) -> 0603WAF1002T5E
Changed lines of the file:
@@
 F 2 "Capacitor_SMD:C_0805_2012Metric" H 4038 2600 50  0001 C CNN
 F 3 "~" H 4000 2750 50  0001 C CNN
-F 4 "CL21B105KBFNNNG" H 4000 2750 50  0001 C CNN "manf#"
+F 4 "CL21B105KBFNNNE" H 4000 2750 50  0001 C CNN "manf#"
+F 5 "C28323" H 0   0   50  0001 C CNN "lcsc#"
 	1    4000 2750
 	1    0    0    -1
@@
 F 2 "Resistor_SMD:R_0603_1608Metric" V 4730 2350 50  0001 C CNN
 F 3 "~" H 4800 2350 50  0001 C CNN
+F 4 "C25804" H 0   0   50  0001 C CNN "lcsc#"
+F 5 "0603WAF1002T5E" H 0   0   50  0001 C CNN "manf#"
 	1    4800 2350
 	-1   0    0    -1
