File: usb.sch (KiCad schematic (older format))
At the start: 11 parts, among them J23 USB_B_Micro, Q3 SS8050, Q4 SS8050, U5 CH340C

Commit message: Added images Added information to schematic Added information to layout
Parts:
- renumbered C30 to C26, C32 to C27, C10 to C28, J23 to J19, R25 to R23, R26 to R24, R27 to R25, R28 to R26
Changed lines of the file:
@@
 encoding utf-8
 Sheet 10 11
-Title ""
-Date ""
-Rev ""
-Comp ""
-Comment1 ""
+Title "AirMon"
+Date "2020-01-13"
+Rev "0.1"
+Comp "Jörg Bayer"
+Comment1 "CC BY 4.0"
 Comment2 ""
 Comment3 ""
@@
 AR Path="/5DD6D4DA/5DEBB035/5E1ECE31" Ref="R?"  Part="1"
 AR Path="/5E1BB661/5E1ECE31" Ref="R?"  Part="1"
-AR Path="/5E1EC3C1/5E1ECE31" Ref="R27"  Part="1"
-F 0 "R27" H 8980 2246 50  0000 R CNN
+AR Path="/5E1EC3C1/5E1ECE31" Ref="R25"  Part="1"
+F 0 "R25" H 8980 2246 50  0000 R CNN
 F 1 "10k" H 8980 2155 50  0000 R CNN
 F 2 "Resistor_SMD:R_0603_1608Metric" V 8980 2200 50  0001 C CNN
@@
 AR Path="/5DD6D4DA/5DEBB035/5E1ECEA6" Ref="R?"  Part="1"
 AR Path="/5E1BB661/5E1ECEA6" Ref="R?"  Part="1"
-AR Path="/5E1EC3C1/5E1ECEA6" Ref="R28"  Part="1"
-F 0 "R28" H 8980 3046 50  0000 R CNN
+AR Path="/5E1EC3C1/5E1ECEA6" Ref="R26"  Part="1"
+F 0 "R26" H 8980 3046 50  0000 R CNN
 F 1 "10k" H 8980 2955 50  0000 R CNN
 F 2 "Resistor_SMD:R_0603_1608Metric" V 8980 3000 50  0001 C CNN
@@
 AR Path="/5DD6D4DA/5DEBB035/5E1EDAED" Ref="R?"  Part="1"
 AR Path="/5E1BB661/5E1EDAED" Ref="R?"  Part="1"
-AR Path="/5E1EC3C1/5E1EDAED" Ref="R25"  Part="1"
-F 0 "R25" H 6580 2746 50  0000 R CNN
+AR Path="/5E1EC3C1/5E1EDAED" Ref="R23"  Part="1"
+F 0 "R23" H 6580 2746 50  0000 R CNN
 F 1 "470R" H 6580 2655 50  0000 R CNN
 F 2 "Resistor_SMD:R_0603_1608Metric" V 6580 2700 50  0001 C CNN
@@
 AR Path="/5DD6D4DA/5DEBB035/5E1EDD07" Ref="R?"  Part="1"
 AR Path="/5E1BB661/5E1EDD07" Ref="R?"  Part="1"
-AR Path="/5E1EC3C1/5E1EDD07" Ref="R26"  Part="1"
-F 0 "R26" H 7180 2646 50  0000 R CNN
+AR Path="/5E1EC3C1/5E1EDD07" Ref="R24"  Part="1"
+F 0 "R24" H 7180 2646 50  0000 R CNN
 F 1 "470R" H 7180 2555 50  0000 R CNN
 F 2 "Resistor_SMD:R_0603_1608Metric" V 7180 2600 50  0001 C CNN
@@
 AR Path="/5E15DEC3/5E1FCEA9" Ref="C?"  Part="1"
 AR Path="/5E151517/5E1FCEA9" Ref="C?"  Part="1"
-AR Path="/5E1EC3C1/5E1FCEA9" Ref="C32"  Part="1"
-F 0 "C32" H 5415 1996 50  0000 L CNN
+AR Path="/5E1EC3C1/5E1FCEA9" Ref="C27"  Part="1"
+F 0 "C27" H 5415 1996 50  0000 L CNN
 F 1 "100n" H 5415 1905 50  0000 L CNN
 F 2 "Capacitor_SMD:C_0603_1608Metric" H 5338 1800 50  0001 C CNN
@@
 AR Path="/5E15DEC3/5E206FF3" Ref="C?"  Part="1"
 AR Path="/5E151517/5E206FF3" Ref="C?"  Part="1"
-AR Path="/5E1EC3C1/5E206FF3" Ref="C30"  Part="1"
-F 0 "C30" H 3615 4096 50  0000 L CNN
+AR Path="/5E1EC3C1/5E206FF3" Ref="C26"  Part="1"
+F 0 "C26" H 3615 4096 50  0000 L CNN
 F 1 "10u" H 3615 4005 50  0000 L CNN
 F 2 "Capacitor_SMD:C_1206_3216Metric" H 3538 3900 50  0001 C CNN
@@
 	3500 4300 3500 4200
 $Comp
-L Connector:USB_B_Micro J23
+L Connector:USB_B_Micro J19
 U 1 1 5E20AD27
 P 3000 2900
-F 0 "J23" H 3055 3367 50  0000 C CNN
+F 0 "J19" H 3055 3367 50  0000 C CNN
 F 1 "USB_B_Micro" H 3055 3276 50  0000 C CNN
 F 2 "global:USB_Micro-B_Molex-105017-0001" H 3150 2850 50  0001 C CNN
@@
 	3000 4300 3500 4300
 $Comp
-L power:VBUS #PWR045
+L power:VBUS #PWR040
 U 1 1 5E211477
 P 3500 2400
-F 0 "#PWR045" H 3500 2250 50  0001 C CNN
+F 0 "#PWR040" H 3500 2250 50  0001 C CNN
 F 1 "VBUS" H 3515 2573 50  0000 C CNN
 F 2 "" H 3500 2400 50  0001 C CNN
@@
 AR Path="/5E1C55BA/5E212E63" Ref="#PWR?"  Part="1"
 AR Path="/5E1CBADF/5E212E63" Ref="#PWR?"  Part="1"
-AR Path="/5E1EC3C1/5E212E63" Ref="#PWR047"  Part="1"
-F 0 "#PWR047" H 5800 4250 50  0001 C CNN
+AR Path="/5E1EC3C1/5E212E63" Ref="#PWR043"  Part="1"
+F 0 "#PWR043" H 5800 4250 50  0001 C CNN
 F 1 "VSS" H 5700 4500 50  0000 C CNN
 F 2 "" H 5800 4400 50  0001 C CNN
@@
 AR Path="/5E1C55BA/5E214237" Ref="#PWR?"  Part="1"
 AR Path="/5E1CBADF/5E214237" Ref="#PWR?"  Part="1"
-AR Path="/5E1EC3C1/5E214237" Ref="#PWR046"  Part="1"
-F 0 "#PWR046" H 5300 2050 50  0001 C CNN
+AR Path="/5E1EC3C1/5E214237" Ref="#PWR041"  Part="1"
+F 0 "#PWR041" H 5300 2050 50  0001 C CNN
 F 1 "VSS" H 5200 2300 50  0000 C CNN
 F 2 "" H 5300 2200 50  0001 C CNN
@@
 AR Path="/5E15DEC3/5E1E42E4" Ref="C?"  Part="1"
 AR Path="/5E151517/5E1E42E4" Ref="C?"  Part="1"
-AR Path="/5E1EC3C1/5E1E42E4" Ref="C10"  Part="1"
-F 0 "C10" H 6315 1996 50  0000 L CNN
+AR Path="/5E1EC3C1/5E1E42E4" Ref="C28"  Part="1"
+F 0 "C28" H 6315 1996 50  0000 L CNN
 F 1 "100n" H 6315 1905 50  0000 L CNN
 F 2 "Capacitor_SMD:C_0603_1608Metric" H 6238 1800 50  0001 C CNN
@@
 AR Path="/5E1C55BA/5E1E42EC" Ref="#PWR?"  Part="1"
 AR Path="/5E1CBADF/5E1E42EC" Ref="#PWR?"  Part="1"
-AR Path="/5E1EC3C1/5E1E42EC" Ref="#PWR015"  Part="1"
-F 0 "#PWR015" H 6200 2050 50  0001 C CNN
+AR Path="/5E1EC3C1/5E1E42EC" Ref="#PWR044"  Part="1"
+F 0 "#PWR044" H 6200 2050 50  0001 C CNN
 F 1 "VSS" H 6100 2300 50  0000 C CNN
 F 2 "" H 6200 2200 50  0001 C CNN
@@
 AR Path="/5E15DEC3/5E1E8B2A" Ref="#PWR?"  Part="1"
 AR Path="/5E151517/5E1E8B2A" Ref="#PWR?"  Part="1"
-AR Path="/5E1EC3C1/5E1E8B2A" Ref="#PWR014"  Part="1"
-F 0 "#PWR014" H 5800 1450 50  0001 C CNN
+AR Path="/5E1EC3C1/5E1E8B2A" Ref="#PWR042"  Part="1"
+F 0 "#PWR042" H 5800 1450 50  0001 C CNN
 F 1 "VCC" H 5817 1773 50  0000 C CNN
 F 2 "" H 5800 1600 50  0001 C CNN

Commit message: Added fuse for USB Added buttons for boot and reset Added version number to PCB Changed several component values for improved manufacturing Added BOM Added component position file
Parts:
- added F1: Polyfuse, Fuse:Fuse_0603_1608Metric, symbol Device:Polyfuse
- C26: lcsc# (none) -> C13585; manf# CL31B106KBHNNNE -> CL31A106KBHNNNE
- C27, C28: lcsc# (none) -> C14663; manf# CL10B104KB8NNNL -> CC0603KRX7R9BB104
- J19: lcsc# (none) -> C136000; manf# (none) -> 105017-0001
- Q3, Q4: lcsc# (none) -> C2150
- R23, R24: lcsc# (none) -> C23179; manf# (none) -> 0603WAF4700T5E
- R25, R26: lcsc# (none) -> C25804; manf# (none) -> 0603WAF1002T5E
- U5: lcsc# (none) -> C84681; manf# (none) -> CH340C
Connections:
- net VBUS: now also F1.1; no longer C26.1, J19.1 (VBUS)
- new net: C26.1, F1.2, J19.1 (VBUS)
Changed lines of the file:
@@
 F 3 "~" H 9500 2200 50  0001 C CNN
 F 4 "SS8050" H 9500 2200 50  0001 C CNN "manf#"
+F 5 "C2150" H 0   0   50  0001 C CNN "lcsc#"
 	1    9500 2200
 	1    0    0    -1
@@
 F 2 "Resistor_SMD:R_0603_1608Metric" V 8980 2200 50  0001 C CNN
 F 3 "~" H 9050 2200 50  0001 C CNN
+F 4 "C25804" H 0   0   50  0001 C CNN "lcsc#"
+F 5 "0603WAF1002T5E" H 0   0   50  0001 C CNN "manf#"
 	1    9050 2200
 	0    -1   -1   0
@@
 F 3 "~" H 9500 3000 50  0001 C CNN
 F 4 "SS8050" H 9500 3000 50  0001 C CNN "manf#"
+F 5 "C2150" H 0   0   50  0001 C CNN "lcsc#"
 	1    9500 3000
 	1    0    0    1
@@
 F 2 "Resistor_SMD:R_0603_1608Metric" V 8980 3000 50  0001 C CNN
 F 3 "~" H 9050 3000 50  0001 C CNN
+F 4 "C25804" H 0   0   50  0001 C CNN "lcsc#"
+F 5 "0603WAF1002T5E" H 0   0   50  0001 C CNN "manf#"
 	1    9050 3000
 	0    -1   1    0
@@
 F 2 "Resistor_SMD:R_0603_1608Metric" V 6580 2700 50  0001 C CNN
 F 3 "~" H 6650 2700 50  0001 C CNN
+F 4 "C23179" H 0   0   50  0001 C CNN "lcsc#"
+F 5 "0603WAF4700T5E" H 0   0   50  0001 C CNN "manf#"
 	1    6650 2700
 	0    -1   -1   0
@@
 F 2 "Resistor_SMD:R_0603_1608Metric" V 7180 2600 50  0001 C CNN
 F 3 "~" H 7250 2600 50  0001 C CNN
+F 4 "C23179" H 0   0   50  0001 C CNN "lcsc#"
+F 5 "0603WAF4700T5E" H 0   0   50  0001 C CNN "manf#"
 	1    7250 2600
 	0    -1   -1   0
@@
 F 2 "Capacitor_SMD:C_0603_1608Metric" H 5338 1800 50  0001 C CNN
 F 3 "~" H 5300 1950 50  0001 C CNN
-F 4 "CL10B104KB8NNNL" H 5300 1950 50  0001 C CNN "manf#"
+F 4 "CC0603KRX7R9BB104" H 5300 1950 50  0001 C CNN "manf#"
+F 5 "C14663" H 0   0   50  0001 C CNN "lcsc#"
 	1    5300 1950
 	1    0    0    -1
@@
 F 2 "Capacitor_SMD:C_1206_3216Metric" H 3538 3900 50  0001 C CNN
 F 3 "~" H 3500 4050 50  0001 C CNN
-F 4 "CL31B106KBHNNNE" H 3500 4050 50  0001 C CNN "manf#"
+F 4 "CL31A106KBHNNNE" H 3500 4050 50  0001 C CNN "manf#"
+F 5 "C13585" H 0   0   50  0001 C CNN "lcsc#"
 	1    3500 4050
 	1    0    0    -1
@@
 F 2 "global:USB_Micro-B_Molex-105017-0001" H 3150 2850 50  0001 C CNN
 F 3 "~" H 3150 2850 50  0001 C CNN
+F 4 "	C136000" H 0   0   50  0001 C CNN "lcsc#"
+F 5 "105017-0001" H 0   0   50  0001 C CNN "manf#"
 	1    3000 2900
 	1    0    0    -1
@@
 L power:VBUS #PWR040
 U 1 1 5E211477
-P 3500 2400
-F 0 "#PWR040" H 3500 2250 50  0001 C CNN
-F 1 "VBUS" H 3515 2573 50  0000 C CNN
-F 2 "" H 3500 2400 50  0001 C CNN
-F 3 "" H 3500 2400 50  0001 C CNN
-	1    3500 2400
+P 3500 2200
+F 0 "#PWR040" H 3500 2050 50  0001 C CNN
+F 1 "VBUS" H 3515 2373 50  0000 C CNN
+F 2 "" H 3500 2200 50  0001 C CNN
+F 3 "" H 3500 2200 50  0001 C CNN
+	1    3500 2200
 	1    0    0    -1
 $EndComp
@@
 F 2 "Package_SO:SOIC-16_3.9x9.9mm_P1.27mm" H 5850 2450 50  0001 L CNN
 F 3 "http://www.datasheet5.com/pdf-local-2195953" H 5450 3800 50  0001 C CNN
+F 4 "C84681" H 0   0   50  0001 C CNN "lcsc#"
+F 5 "CH340C" H 0   0   50  0001 C CNN "manf#"
 	1    5800 3000
 	1    0    0    -1
@@
 NoConn ~ 6200 2900
 Wire Wire Line
-	3500 2400 3500 2700
+	3500 2600 3500 2700
 Wire Wire Line
 	5800 3600 5800 4300
@@
 F 2 "Capacitor_SMD:C_0603_1608Metric" H 6238 1800 50  0001 C CNN
 F 3 "~" H 6200 1950 50  0001 C CNN
-F 4 "CL10B104KB8NNNL" H 6200 1950 50  0001 C CNN "manf#"
+F 4 "CC0603KRX7R9BB104" H 6200 1950 50  0001 C CNN "manf#"
+F 5 "C14663" H 0   0   50  0001 C CNN "lcsc#"
 	1    6200 1950
 	-1   0    0    -1
@@
 Wire Wire Line
 	6200 2600 7100 2600
+$Comp
+L Device:Polyfuse F1
+U 1 1 5E1F9E89
+P 3500 2450
+F 0 "F1" H 3588 2496 50  0000 L CNN
+F 1 "Polyfuse" H 3588 2405 50  0000 L CNN
+F 2 "Fuse:Fuse_0603_1608Metric" H 3550 2250 50  0001 L CNN
+F 3 "~" H 3500 2450 50  0001 C CNN
+F 4 "0603L050SLYR" H 3500 2450 50  0001 C CNN "manf#"
+F 5 "C207014" H 0   0   50  0001 C CNN "lcsc#"
+	1    3500 2450
+	1    0    0    -1
+$EndComp
+Wire Wire Line
+	3500 2200 3500 2300
 $EndSCHEMATC
